File: eagle/attenuverter.sch (EAGLE design)
At the start: 6 parts, among them IC1 TL082P, U1 POWER

Commit message: schemo done
Parts:
- removed U$1, U$2: AUDIO-JACK, erthenvar:AUDIO-JACK
- added ADJ: 100k, pot:3RP/1610N
- added CV_IN, CV_OUT: AUDIO-JACK, erthenvar:AUDIO-JACK
- added LED1: NEG, SparkFun-LED:LED5MM
- added LED2: POS, SparkFun-LED:LED5MM
- added R1: 330, rcl:R-US_0207/10
- added R2: 4k7, rcl:R-US_0207/10
- added R3, R4: 220k, rcl:R-US_0207/10
- added R6: 680, rcl:R-US_0207/10
- added R7: 100k, rcl:R-US_0207/10
- C1, C2: value (none) -> 10n
Connections:
- new net N$11: CV_IN.NORM, R7.1
- new net N$2: ADJ.E, CV_IN.TIP, R3.1
- new net N$3: IC1A.-IN, R3.2, R4.1
- new net N$4: IC1A.OUT, IC1B.+IN, R1.1, R4.2
- new net N$5: CV_OUT.TIP, R1.2
- new net N$6: ADJ.S, IC1A.+IN
- new net N$7: IC1B.OUT, LED1.C, LED2.A
- new net N$8: LED1.A, LED2.C, R2.2, R6.2
- new net N$9: IC1B.-IN, R2.1
- net +12V: now also R7.2
- net GND: now also ADJ.A, CV_IN.RING, CV_OUT.RING, R6.1
Other:
- moved on the sheet: C1, C2, IC1A, IC1B, U1

Commit message: routed
Connections:
- net GND: now also ADJ.E; no longer ADJ.A
- net N$2: now also ADJ.A; no longer ADJ.E
Other:
- moved on the sheet: ADJ
Changed lines of the file:
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@@
 <instance part="GND3" gate="1" x="12.7" y="55.88"/>
 <instance part="GND4" gate="1" x="86.36" y="55.88"/>
-<instance part="ADJ" gate="G$1" x="25.4" y="66.04"/>
+<instance part="ADJ" gate="G$1" x="25.4" y="66.04" rot="MR180"/>
 <instance part="R6" gate="G$1" x="104.14" y="25.4" rot="R90"/>
 <instance part="GND5" gate="1" x="104.14" y="15.24"/>
@@
 </segment>
 <segment>
-<pinref part="ADJ" gate="G$1" pin="A"/>
 <pinref part="GND6" gate="1" pin="GND"/>
+<pinref part="ADJ" gate="G$1" pin="E"/>
 <wire x1="25.4" y1="58.42" x2="25.4" y2="60.96" width="0.1524" layer="91"/>
 </segment>
@@
 <pinref part="CV_IN" gate="G$1" pin="TIP"/>
 <wire x1="12.7" y1="73.66" x2="25.4" y2="73.66" width="0.1524" layer="91"/>
-<pinref part="ADJ" gate="G$1" pin="E"/>
+<pinref part="ADJ" gate="G$1" pin="A"/>
 <wire x1="25.4" y1="73.66" x2="30.48" y2="73.66" width="0.1524" layer="91"/>
 <wire x1="25.4" y1="71.12" x2="25.4" y2="73.66" width="0.1524" layer="91"/>
